File: PicoIO-THT/PicoIO-THT.kicad_pcb (KiCad board)
At the start: 2 copper layers, 73.2 x 58.4 mm, 52 parts, among them J1 Conn_01x04, J10 Conn_01x04, J11 Conn_01x03, J12 Conn_01x06, J14 Conn_01x02, J2 Conn_01x04, J3 Conn_01x04, J4 Conn_01x04, J5 Conn_01x04, J6 Conn_01x04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

Commit message: Remove leftover vias
Routing:
- net P1 CN LED: track 9.27 -> 9.45 mm, vias 1 -> 0
- net P1 UL LED: track 9.07 -> 9.26 mm, vias 1 -> 0
Changed lines of the file:
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@@
   (segment (start 127.232 96.371) (end 127.232 93.655) (width 0.25) (layer "F.Cu") (net 4))
   (segment (start 128.143 105.345) (end 128.143 97.282) (width 0.25) (layer "F.Cu") (net 4))
-  (segment (start 125.73 100.584) (end 124.692 99.546) (width 0.25) (layer "F.Cu") (net 5))
-  (segment (start 124.692 99.546) (end 124.692 93.655) (width 0.25) (layer "F.Cu") (net 5))
-  (via (at 125.73 100.584) (size 0.8) (drill 0.4) (layers "F.Cu" "B.Cu") (net 5))
+  (segment (start 126.815 101.85) (end 124.692 99.727) (width 0.25) (layer "F.Cu") (net 5))
+  (segment (start 124.692 99.727) (end 124.692 93.655) (width 0.25) (layer "F.Cu") (net 5))
   (segment (start 126.815 101.85) (end 126.815 101.669) (width 0.25) (layer "B.Cu") (net 5))
-  (segment (start 126.815 101.669) (end 125.73 100.584) (width 0.25) (layer "B.Cu") (net 5))
   (segment (start 141.6 98.039) (end 139.932 96.371) (width 0.25) (layer "F.Cu") (net 6))
   (segment (start 140.48 106.508) (end 141.6 105.388) (width 0.25) (layer "F.Cu") (net 6))
   (segment (start 139.932 96.371) (end 139.932 93.655) (width 0.25) (layer "F.Cu") (net 6))
   (segment (start 141.6 105.388) (end 141.6 98.039) (width 0.25) (layer "F.Cu") (net 6))
-  (segment (start 139.2075 100.584) (end 137.392 98.7685) (width 0.25) (layer "F.Cu") (net 7))
-  (segment (start 137.392 98.7685) (end 137.392 93.655) (width 0.25) (layer "F.Cu") (net 7))
-  (via (at 139.2075 100.584) (size 0.8) (drill 0.4) (layers "F.Cu" "B.Cu") (net 7))
-  (segment (start 140.33 101.7065) (end 139.2075 100.584) (width 0.25) (layer "B.Cu") (net 7))
+  (segment (start 140.425 101.85) (end 137.392 98.817) (width 0.25) (layer "F.Cu") (net 7))
+  (segment (start 137.392 98.817) (end 137.392 93.655) (width 0.25) (layer "F.Cu") (net 7))
   (segment (start 152.632 105.16) (end 153.98 106.508) (width 0.25) (layer "F.Cu") (net 8))
   (segment (start 152.632 93.655) (end 152.632 105.16) (width 0.25) (layer "F.Cu") (net 8))
